File: Hardware/WCH-Eth-Base/WCH-Eth-Base-Power.kicad_sch (KiCad schematic)
At the start: 16 parts, among them IC2 RY8310, J6 Conn_01x02_Pin, Q1 AO3401A

Commit message: add Files and First Layout things
Parts:
- removed C24, C27, C28: 22u, Capacitor_SMD:CP_Elec_5x5.4, symbol Device:C_Polarized
- removed D12: 15V, Diode_SMD:D_SOD-323, symbol Device:D_Zener
- removed D13: PWR, symbol Device:LED
- removed J6: Conn_01x02_Pin, Connector_JST:JST_PH_B2B-PH-SM4-TB_1x02-1MP_P2.00mm_Vertical, symbol Connector:Conn_01x02_Pin
- removed Q1: AO3401A, Package_TO_SOT_SMD:TSOT-23, symbol Transistor_FET:AO3401A
- removed R19: 100k, Resistor_SMD:R_0402_1005Metric, symbol Device:R
- added C15: 22u, Capacitor_SMD:CP_Elec_5x5.4, symbol Device:C_Polarized
- added C18, C46: 22u, Capacitor_SMD:C_0402_1005Metric, symbol Device:C
- added D12, D14: D_Schottky, Diode_SMD:D_SMA, symbol Device:D_Schottky
- added D13: LED_ARGB, LCSC:LED-ARRAY-SMD_MHS110FRGBCT, symbol Device:LED_ARGB
- added R21, R23: 1k, Resistor_SMD:R_0402_1005Metric, symbol Device:R
- R22: value R -> 1k
- renumbered C23 to C14, C25 to C16, C26 to C17, IC2 to IC3, L2 to L1, R20 to R19, R21 to R20
Connections:
- net +3.3V: now also C18.1, D13.1 (A); no longer R22.1
- net GND: now also R22.2, C15.2, C18.2, C46.2, R21.2, R23.2
- net VCC: now also C14.1, IC3.4 (EN), IC3.5 (IN), C15.1, C46.1, D12.1 (K), D14.1 (K)
- new net: D13.2 (RK), R21.1
- new net: D13.3 (GK), R22.1
- new net: D13.4 (BK), R23.1
- new net +12V: D14.2 (A)
- new net VBUS: D12.2 (A)
