File: Hardware/WCH-Eth-Base/WCH-Eth-Base-eth.kicad_sch (KiCad schematic)
At the start: 28 parts, among them U4 RT9400

Commit message: add Files and First Layout things
Parts:
- removed C14, C19, C22: 1000pF/2KV, symbol Device:C
- removed C15, C16, C17, C18, C20, C21: 100n, Capacitor_SMD:C_0402_1005Metric, symbol Device:C
- removed L1: G48C01S, LCSC:SMD-48_L27.8-W12.3-P1.02-LS15.3-BL, symbol LCSC:G48C01S
- removed R10, R11, R12, R13, R14, R15, R16, R17: 75, Resistor_SMD:R_0402_1005Metric, symbol Device:R
- removed R18: R, Capacitor_SMD:C_1206_3216Metric, symbol Device:R
- removed R23, R24, R25, R27: R_Small, symbol Device:R_Small
- removed RJ1: KH-56-8P8C-1X2-D, LCSC:RJ45-TH_KH-56-8P8C-1X2-D, symbol LCSC:KH-56-8P8C-1X2-D
- removed U4: RT9400, Techbeard:RT9400, symbol Techbeard:RT9400
- added C31, C32, C33, C34, C35, C36, C37, C38, C39, C40, C41, C42, C43, C44, C45: 100n, Capacitor_SMD:C_0402_1005Metric, symbol Device:C
- added R16, R17: 4k7, Resistor_SMD:R_0402_1005Metric, symbol Device:R_Small
- added Y2: Crystal_GND24, Crystal:Crystal_SMD_3225-4Pin_3.2x2.5mm, symbol Device:Crystal_GND24
- C12, C13: value 100n -> C
Connections:
- net +3.3V: now also IC1.14 (AVDDH), IC1.19 (AVDDL), IC1.24 (AVDDH), IC1.27 (AVDDL), IC1.29 (AVDDH), IC1.3 (AVDDH), IC1.31 (DVDDL), IC1.34 (AVDDL), IC1.37 (AVDDH), IC1.39 (DVDDL), IC1.40 (DVDDIO_1), IC1.54 (DVDDIO_1), IC1.63 (DVDDIO), IC1.64 (DVDDL), IC1.73 (AVDDH), IC1.8 (AVDDL), C31.1, C32.1, C33.1, C34.1, C35.1, C36.1, C37.1, C38.1, C39.1, C40.1, C41.1, C42.1, C43.1, C44.1, C45.1, R16.1, R17.1
- net ETH_SCK: now also R16.2
- net ETH_SDA: now also R17.2
- net Eth0_LedL: now also IC1.68 (GPO47/P1LED2/SMI_SEL_1)
- net Eth0_LedR: now also IC1.70 (GPIO49/P1LED1)
- net Eth1_LedL: now also IC1.65 (GPIO44/P3LED2)
- net Eth1_LedR: now also IC1.67 (GPIO46/P3LED1)
- net GND: now also C12.2, C13.2, IC1.25 (AGND), IC1.56 (GND_SWR), IC1.57 (GND_SWR), IC1.77 (EP), C31.2, C32.2, C33.2, C34.2, C35.2, C36.2, C37.2, C38.2, C39.2, C40.2, C41.2, C42.2, C43.2, C44.2, C45.2, Y2.2, Y2.4
- net P1MDICN: now reaches IC1.10 (P1MDICN)
- net P1MDIDP: now reaches IC1.11 (P1MDIDP)
- net P1MDIDN: now reaches IC1.12 (P1MDIDN)
- net P2MDIAP: now reaches IC1.15 (P3MDIAP)
- net P2MDIAN: now reaches IC1.16 (P3MDIAN)
- net P2MDIBP: now reaches IC1.17 (P3MDIBP)
- net P2MDIBN: now reaches IC1.18 (P3MDIBN)
- net P2MDICP: now reaches IC1.20 (P3MDICP)
- net P2MDICN: now reaches IC1.21 (P3MDICN)
- net P2MDIDP: now reaches IC1.22 (P3MDIDP)
- net P2MDIDN: now reaches IC1.23 (P3MDIDN)
- net P1MDIAP: now reaches IC1.4 (P1MDIAP)
- net P1MDIAN: now reaches IC1.5 (P1MDIAN)
- net P1MDIBP: now reaches IC1.6 (P1MDIBP)
- net P1MDIBN: now reaches IC1.7 (P1MDIBN)
- net at IC1.74 (XTALO): now also C12.1, Y2.1
- net at IC1.75 (XTALI): now also C13.1, Y2.3
- net P1MDICP: now reaches IC1.9 (P1MDICP)
- no-connect marks 0 -> 5
Other:
- added sheet Ethernet Mag+RJ45 (WCH-Eth-Base-EthMag.kicad_sch)
- moved on the sheet: IC1
