File: Hardware/WCH-Eth-Base/WCH-Eth-Base.kicad_pcb (KiCad board)
At the start: 4 copper layers, 99.9 x 50 mm, 72 parts, among them IC2 RY8310, J3 USB_C_Receptacle_USB2.0, J4 USB_C_Receptacle_USB2.0, J7 Conn_02x32_Counter_Clockwise, Q1 AO3401A, SW3 RotaryEncoder_Switch, U1 CH32V307VCT6, U2 WE-TVS-82400102, U3 WE-TVS-82400102, U4 RT9400, Y1 Crystal_GND24

Commit message: add Files and First Layout things
Parts:
- removed IC2: RY8310, Package_TO_SOT_SMD:SOT-23-6
- removed J3: USB_C_Receptacle_USB2.0, LCSC:TYPE-C-TH_TYPE-C-14P-CC-2.6
- removed Q1: AO3401A, Package_TO_SOT_SMD:TSOT-23
- removed R18: R, Capacitor_SMD:C_1206_3216Metric
- added C14: 100n, Capacitor_SMD:C_0402_1005Metric, B.Cu at (154.3, 44.2)
- added C19: 22u, Capacitor_SMD:CP_Elec_5x5.4, F.Cu at (160.7, 50.4)
- added C22: 1000pF/2KV, Capacitor_SMD:C_1206_3216Metric, B.Cu at (123.3, 66.5)
- added C29: 100n, Capacitor_SMD:C_0402_1005Metric, B.Cu at (140.1, 71.9)
- added C30: 1000pF/2KV, Capacitor_SMD:C_1206_3216Metric, B.Cu at (112.2, 63.5)
- added C31: 100n, Capacitor_SMD:C_0402_1005Metric, B.Cu at (134.4, 52.3)
- added C32: 100n, Capacitor_SMD:C_0402_1005Metric, B.Cu at (127.9, 54.7)
- added C33: 100n, Capacitor_SMD:C_0402_1005Metric, B.Cu at (124.6, 52.5)
- added C34: 100n, Capacitor_SMD:C_0402_1005Metric, B.Cu at (122.3, 50.3)
- added C35: 100n, Capacitor_SMD:C_0402_1005Metric, B.Cu at (105.4, 47.4)
- added C36: 100n, Capacitor_SMD:C_0402_1005Metric, B.Cu at (105.4, 49.1)
- added C37: 100n, Capacitor_SMD:C_0402_1005Metric, B.Cu at (103.1, 40.8)
- added C38: 100n, Capacitor_SMD:C_0402_1005Metric, B.Cu at (103.1, 42.5)
- added C39: 100n, Capacitor_SMD:C_0402_1005Metric, B.Cu at (130.8, 55.9)
- added C40: 100n, Capacitor_SMD:C_0402_1005Metric, B.Cu at (125.4, 53.3)
- added C41: 100n, Capacitor_SMD:C_0402_1005Metric, B.Cu at (123.9, 51.8)
- added C42: 100n, Capacitor_SMD:C_0402_1005Metric, B.Cu at (123.1, 51.0)
- added C43: 100n, Capacitor_SMD:C_0402_1005Metric, B.Cu at (100.9, 40.8)
- added C44: 100n, Capacitor_SMD:C_0402_1005Metric, B.Cu at (121.6, 49.5)
- added C45: 100n, Capacitor_SMD:C_0402_1005Metric, B.Cu at (100.9, 44.1)
- added C46: 22u, Capacitor_SMD:C_0402_1005Metric, F.Cu at (148.1, 67.1)
- added C48: 22u, Capacitor_SMD:CP_Elec_5x5.4, F.Cu at (160.7, 56.4)
- added D10: D_Schottky, Diode_SMD:D_SMA, F.Cu at (124.7, 27.7)
- added D11: D_Schottky, Diode_SMD:D_SMA, F.Cu at (134.3, 18.9)
- added D13: LED_ARGB, LCSC:LED-ARRAY-SMD_MHS110FRGBCT, B.Cu at (146.9, 85.8)
- added D3: LED_ARGB, LCSC:LED-ARRAY-SMD_MHS110FRGBCT, B.Cu at (159.5, 85.8)
- added D4: D_TVS, Diode_SMD:D_SMA, F.Cu at (166.3, 91.2)
- added IC3: RY8310, Package_TO_SOT_SMD:SOT-23-6, B.Cu at (151.5, 45.2)
- added J5: USB_C_Receptacle_USB2.0, LCSC:TYPE-C-TH_TYPE-C-14P-CC-2.6, F.Cu at (149.8, 79.9)
- added J6: Conn_ARM_SWD_TagConnect_TC2030-NL, Connector:Tag-Connect_TC2030-IDC-NL_2x03_P1.27mm_Vertical, F.Cu at (169.3, 70.7)
- added R23: 1k, Resistor_SMD:R_0402_1005Metric, B.Cu at (148.1, 84.3)
- added R24: 49k9, Resistor_SMD:R_0402_1005Metric, B.Cu at (118.7, 60.3)
- added R25: 49k9, Resistor_SMD:R_0402_1005Metric, B.Cu at (121.8, 60.3)
- added R27: 49k9, Resistor_SMD:R_0402_1005Metric, B.Cu at (127.9, 60.3)
- added R33: 75, Resistor_SMD:R_0402_1005Metric, B.Cu at (121.8, 69.7)
- added R34: 75, Resistor_SMD:R_0402_1005Metric, B.Cu at (124.8, 69.7)
- added R35: 75, Resistor_SMD:R_0402_1005Metric, B.Cu at (127.9, 69.7)
- added R36: 75, Resistor_SMD:R_0402_1005Metric, B.Cu at (130.9, 69.7)
- added R37: 75, Resistor_SMD:R_0402_1005Metric, B.Cu at (134.0, 69.7)
- added R38: 75, Resistor_SMD:R_0402_1005Metric, B.Cu at (137.1, 69.7)
- added R39: 75, Resistor_SMD:R_0402_1005Metric, B.Cu at (140.1, 69.7)
- added R40: R, Capacitor_SMD:C_1206_3216Metric, B.Cu at (109.5, 63.5)
- added R41: R_Small, Resistor_SMD:R_0402_1005Metric, B.Cu at (114.1, 77.2)
- added R42: R_Small, Resistor_SMD:R_0402_1005Metric, B.Cu at (125.5, 77.2)
- added R43: R_Small, Resistor_SMD:R_0402_1005Metric, B.Cu at (129.9, 77.2)
- added R44: R_Small, Resistor_SMD:R_0402_1005Metric, B.Cu at (141.3, 77.2)
- added SW1: SW_Push, LCSC:SW-SMD_4P-L5.1-W5.1-P3.70-LS6.5-TL-2, F.Cu at (168.9, 77.8)
- added SW2: SW_Push, LCSC:SW-SMD_4P-L5.1-W5.1-P3.70-LS6.5-TL-2, F.Cu at (175.3, 77.8)
- added Y2: Crystal_GND24, Crystal:Crystal_SMD_3225-4Pin_3.2x2.5mm, B.Cu at (141.7, 46.4)
- C1: value C -> 100n
- C12, C13, C2: value 100n -> C
- C15: value 100n -> 22u; footprint Capacitor_SMD:C_0402_1005Metric -> Capacitor_SMD:CP_Elec_5x5.4; moved to F.Cu
- C18: value 100n -> 22u; moved to F.Cu
- C24, C28: value 22u -> 100n; footprint Capacitor_SMD:CP_Elec_5x5.4 -> Capacitor_SMD:C_0402_1005Metric; moved to B.Cu
- C27: value 22u -> 1000pF/2KV; footprint Capacitor_SMD:CP_Elec_5x5.4 -> Capacitor_SMD:C_1206_3216Metric; moved to B.Cu
- D12: value 15V -> D_Schottky; footprint Diode_SMD:D_SOD-323 -> Diode_SMD:D_SMA; moved to F.Cu
- D14: value LED_ARGB -> D_Schottky; footprint LCSC:LED-ARRAY-SMD_MHS110FRGBCT -> Diode_SMD:D_SMA
- L1: value G48C01S -> 4.7u; footprint LCSC:SMD-48_L27.8-W12.3-P1.02-LS15.3-BL -> Techbeard:L_0630; moved to B.Cu
- L2: value 4.7u -> G48C01S; footprint Techbeard:L_0630 -> LCSC:SMD-48_L27.8-W12.3-P1.02-LS15.3-BL; moved to F.Cu
- R10: value 75 -> 1k
- R11, R16, R17: value 75 -> 4k7
- R12, R13, R14, R15: value 75 -> 5k1
- R19: value 100k -> 31.25 k
- R20: value 31.25 k -> 10k
- R21: value 10k -> 1k
- R22, R6, R7, R9: value R -> 1k
- R26, R28, R29, R30, R31: value 1k -> 49k9
- R32: value 1k -> 75
- R4, R5: value 4k7 -> 1k
- R8: value R -> 4k7
- SW3: footprint Rotary_Encoder:RotaryEncoder_Alps_EC11E-Switch_Vertical_H20mm_CircularMountingHoles -> Techbeard:STEC11B09
- moved R19 127.3 mm to (152.7, 42.8), turned to 0 degrees
- moved R10 126.2 mm to (160.7, 84.3), turned to 90 degrees
- moved R20 125.4 mm to (150.5, 42.8), turned to 0 degrees
- moved R22 122.1 mm to (147.0, 84.3), turned to 90 degrees
- moved C18 121.7 mm to (160.2, 66.3), turned to 0 degrees
- moved R21 121.3 mm to (145.9, 84.3), turned to 90 degrees
- moved R13 120.7 mm to (158.2, 80.1), turned to 90 degrees
- moved R12 118.2 mm to (155.1, 80.0), turned to -90 degrees
- moved C15 113.1 mm to (152.6, 50.4)
- moved R15 113.1 mm to (151.6, 79.9), turned to 90 degrees
- moved C16 111.8 mm to (151.4, 47.6), turned to 0 degrees
- moved R14 110.4 mm to (148.2, 79.9), turned to -90 degrees
- moved C26 106.5 mm to (134.0, 71.9), turned to 90 degrees
- moved C12 105.2 mm to (144.6, 46.7), turned to 90 degrees
- moved C25 103.5 mm to (130.9, 71.9), turned to 90 degrees
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- renumbered J7 to J1
Connections:
- C1 pad 1: Net-(U1-OSC_IN) -> GND
- C1 pad 2: GND -> nRst
- C12 pad 1: Net-(C12-Pad1) -> Net-(IC1-XTALO)
- C12 pad 2: Net-(C12-Pad2) -> GND
- C13 pad 1: Net-(C13-Pad1) -> Net-(IC1-XTALI)
- C13 pad 2: Net-(C13-Pad2) -> GND
- C15 pad 1: Net-(C15-Pad1) -> VCC
- C15 pad 2: Net-(C15-Pad2) -> GND
- C16 pad 1: Net-(C16-Pad1) -> Net-(IC3-CB)
- C16 pad 2: Net-(C16-Pad2) -> Net-(IC3-SW)
- C17 pad 1: Net-(C17-Pad1) -> +3.3V
- C17 pad 2: Net-(C17-Pad2) -> GND
- C18 pad 1: Net-(C18-Pad1) -> +3.3V
- C18 pad 2: Net-(C18-Pad2) -> GND
- C2 pad 1: GND -> Net-(U1-OSC_IN)
- C2 pad 2: nRst -> GND
- C23 pad 1: Net-(D12-K) -> Net-(C23-Pad1)
- C23 pad 2: GND -> Net-(C23-Pad2)
- C24 pad 1: Net-(D12-K) -> Net-(C24-Pad1)
- C24 pad 2: GND -> Net-(C24-Pad2)
- C25 pad 1: Net-(IC2-CB) -> Net-(C25-Pad1)
- C25 pad 2: Net-(IC2-SW) -> Net-(C25-Pad2)
- C26 pad 1: +3.3V -> Net-(C26-Pad1)
- C26 pad 2: GND -> Net-(C26-Pad2)
- C27 pad 1: +3.3V -> Net-(C27-Pad1)
- C27 pad 2: GND -> Earth
- C28 pad 1: +3.3V -> Net-(C28-Pad1)
- C28 pad 2: GND -> Net-(C28-Pad2)
- D12 pad 1: Net-(D12-K) -> VCC
- D12 pad 2: Net-(D12-A) -> VBUS
- D14 pad 1: +3.3V -> VCC
- D14 pad 2: Net-(D14-RK) -> +12V
- IC1 pad 10: unconnected-(IC1-P1MDICN-Pad10) -> P1MDICN
- IC1 pad 11: unconnected-(IC1-P1MDIDP-Pad11) -> P1MDIDP
- IC1 pad 12: unconnected-(IC1-P1MDIDN-Pad12) -> P1MDIDN
- IC1 pad 14: unconnected-(IC1-AVDDH-Pad14) -> +3.3V
- IC1 pad 15: unconnected-(IC1-P3MDIAP-Pad15) -> P2MDIAP
- IC1 pad 16: unconnected-(IC1-P3MDIAN-Pad16) -> P2MDIAN
- IC1 pad 17: unconnected-(IC1-P3MDIBP-Pad17) -> P2MDIBP
- IC1 pad 18: unconnected-(IC1-P3MDIBN-Pad18) -> P2MDIBN
- IC1 pad 19: unconnected-(IC1-AVDDL-Pad19) -> +3.3V
- IC1 pad 20: unconnected-(IC1-P3MDICP-Pad20) -> P2MDICP
- IC1 pad 21: unconnected-(IC1-P3MDICN-Pad21) -> P2MDICN
- IC1 pad 22: unconnected-(IC1-P3MDIDP-Pad22) -> P2MDIDP
- IC1 pad 23: unconnected-(IC1-P3MDIDN-Pad23) -> P2MDIDN
- IC1 pad 24: unconnected-(IC1-AVDDH-Pad24) -> +3.3V
- IC1 pad 25: unconnected-(IC1-AGND-Pad25) -> GND
- IC1 pad 27: unconnected-(IC1-AVDDL-Pad27) -> +3.3V
- IC1 pad 29: unconnected-(IC1-AVDDH-Pad29) -> +3.3V
- IC1 pad 3: unconnected-(IC1-AVDDH-Pad3) -> +3.3V
- IC1 pad 31: unconnected-(IC1-DVDDL-Pad31) -> +3.3V
- IC1 pad 34: unconnected-(IC1-AVDDL-Pad34) -> +3.3V
- IC1 pad 37: unconnected-(IC1-AVDDH-Pad37) -> +3.3V
- IC1 pad 39: unconnected-(IC1-DVDDL-Pad39) -> +3.3V
- IC1 pad 4: unconnected-(IC1-P1MDIAP-Pad4) -> P1MDIAP
- IC1 pad 40: unconnected-(IC1-DVDDIO_1-Pad40) -> +3.3V
- IC1 pad 5: unconnected-(IC1-P1MDIAN-Pad5) -> P1MDIAN
- IC1 pad 54: unconnected-(IC1-DVDDIO_1-Pad54) -> +3.3V
- IC1 pad 56: unconnected-(IC1-GND_SWR-Pad56) -> GND
- IC1 pad 57: unconnected-(IC1-GND_SWR-Pad57) -> GND
- IC1 pad 6: unconnected-(IC1-P1MDIBP-Pad6) -> P1MDIBP
- IC1 pad 63: unconnected-(IC1-DVDDIO-Pad63) -> +3.3V
- IC1 pad 64: unconnected-(IC1-DVDDL-Pad64) -> +3.3V
- IC1 pad 65: unconnected-(IC1-GPIO44/P3LED2-Pad65) -> Eth1_LedL
- IC1 pad 67: unconnected-(IC1-GPIO46/P3LED1-Pad67) -> Eth1_LedR
- IC1 pad 68: unconnected-(IC1-GPO47/P1LED2/SMI_SEL_1-Pad68) -> Eth0_LedL
- IC1 pad 7: unconnected-(IC1-P1MDIBN-Pad7) -> P1MDIBN
- IC1 pad 70: unconnected-(IC1-GPIO49/P1LED1-Pad70) -> Eth0_LedR
- IC1 pad 73: unconnected-(IC1-AVDDH-Pad73) -> +3.3V
- IC1 pad 74: unconnected-(IC1-XTALO-Pad74) -> Net-(IC1-XTALO)
- IC1 pad 75: unconnected-(IC1-XTALI-Pad75) -> Net-(IC1-XTALI)
- IC1 pad 77: unconnected-(IC1-EP-Pad77) -> GND
- IC1 pad 8: unconnected-(IC1-AVDDL-Pad8) -> +3.3V
- IC1 pad 9: unconnected-(IC1-P1MDICP-Pad9) -> P1MDICP
- L1 pad 1: unconnected-(L1-Pad1) -> Net-(IC3-SW)
- L1 pad 2: unconnected-(L1-Pad2) -> +3.3V
- L2 pad 1: Net-(IC2-SW) -> Net-(L2-Pad1)
- L2 pad 2: +3.3V -> P1MDIAP
- R1 pad 2: StateLED1 -> StateLED0
- R10 pad 1: Net-(C12-Pad2) -> Net-(D3-BK)
- R10 pad 2: Net-(C14-Pad1) -> StateLED2
- R11 pad 1: Net-(C13-Pad2) -> +3.3V
- R11 pad 2: Net-(C14-Pad1) -> nRst
- R12 pad 1: Net-(C15-Pad2) -> GND
- R12 pad 2: Net-(C14-Pad1) -> Net-(J4-CC1)
- R13 pad 1: Net-(C16-Pad2) -> GND
- R13 pad 2: Net-(C14-Pad1) -> Net-(J4-CC2)
- R14 pad 1: Net-(C17-Pad2) -> GND
- R14 pad 2: Net-(C19-Pad1) -> Net-(J5-CC1)
- R15 pad 1: Net-(C18-Pad2) -> GND
- R15 pad 2: Net-(C19-Pad1) -> Net-(J5-CC2)
- R16 pad 1: Net-(C20-Pad2) -> +3.3V
- R16 pad 2: Net-(C19-Pad1) -> ETH_SCK
- R17 pad 1: Net-(C21-Pad2) -> +3.3V
- R17 pad 2: Net-(C19-Pad1) -> ETH_SDA
- R19 pad 1: Net-(D12-A) -> Net-(IC3-FB)
- R19 pad 2: GND -> +3.3V
- R2 pad 2: StateLED1 -> StateLED0
- R20 pad 1: Net-(IC2-FB) -> GND
- R20 pad 2: +3.3V -> Net-(IC3-FB)
- R21 pad 1: GND -> Net-(D13-RK)
- R21 pad 2: Net-(IC2-FB) -> GND
- R22 pad 1: +3.3V -> Net-(D13-GK)
- R22 pad 2: Net-(D13-A) -> GND
- R26 pad 1: Net-(D14-GK) -> +3.3V
- R26 pad 2: StateLED2 -> Net-(L2-Pad16)
- R28 pad 1: Net-(D14-RK) -> +3.3V
- R28 pad 2: StateLED2 -> Net-(L2-Pad10)
- R29 pad 1: Net-(D1-BK) -> +3.3V
- R29 pad 2: StateLED1 -> Net-(L2-Pad7)
- R3 pad 1: Net-(D14-BK) -> Net-(D1-BK)
- R3 pad 2: StateLED2 -> StateLED0
- R30 pad 1: Net-(D2-RK) -> +3.3V
- R30 pad 2: StateLED0 -> Net-(L2-Pad4)
- R31 pad 1: Net-(D2-GK) -> +3.3V
- R31 pad 2: StateLED0 -> Net-(L2-Pad1)
- R32 pad 1: Net-(D2-BK) -> Net-(C20-Pad2)
- R32 pad 2: StateLED0 -> Net-(C22-Pad1)
- R4 pad 1: Net-(U1-BOOT0) -> Net-(D2-RK)
- R4 pad 2: GND -> StateLED1
- R5 pad 1: +3.3V -> Net-(D2-GK)
- R5 pad 2: nRst -> StateLED1
- R6 pad 1: GND -> Net-(D2-BK)
- R6 pad 2: Net-(J3-CC1) -> StateLED1
- R7 pad 1: GND -> Net-(D3-RK)
- R7 pad 2: Net-(J3-CC2) -> StateLED2
- R8 pad 1: GND -> Net-(U1-BOOT0)
- R8 pad 2: Net-(J4-CC1) -> GND
- R9 pad 1: GND -> Net-(D3-GK)
- R9 pad 2: Net-(J4-CC2) -> StateLED2
- RJ1 pad 1: Net-(L1-Pad47) -> Eth0_BI_DA+
- RJ1 pad 13: Net-(L1-Pad35) -> Eth1_BI_DA+
- RJ1 pad 14: Net-(L1-Pad34) -> Eth1_BI_DA-
- RJ1 pad 15: Net-(L1-Pad32) -> Eth1_BI_DB+
- RJ1 pad 16: Net-(L1-Pad29) -> Eth1_BI_DC+
- RJ1 pad 17: Net-(L1-Pad28) -> Eth1_BI_DC-
- RJ1 pad 18: Net-(L1-Pad31) -> Eth1_BI_DB-
- RJ1 pad 19: Net-(L1-Pad26) -> Eth1_BI_DD+
- RJ1 pad 2: Net-(L1-Pad46) -> Eth0_BI_DA-
- RJ1 pad 20: Net-(L1-Pad25) -> Eth1_BI_DD-
- RJ1 pad 3: Net-(L1-Pad44) -> Eth0_BI_DB+
- RJ1 pad 4: Net-(L1-Pad41) -> Eth0_BI_DC+
- RJ1 pad 5: Net-(L1-Pad40) -> Eth0_BI_DC-
- RJ1 pad 6: Net-(L1-Pad43) -> Eth0_BI_DB-
- RJ1 pad 7: Net-(L1-Pad38) -> Eth0_BI_DD+
- RJ1 pad 8: Net-(L1-Pad37) -> Eth0_BI_DD-
- SW3 pad A: unconnected-(SW3-PadA) -> EncoderA
- SW3 pad B: unconnected-(SW3-PadB) -> EncoderB
- SW3 pad C: unconnected-(SW3-PadC) -> GND
- SW3 pad S1: unconnected-(SW3-PadS1) -> EncoderS1
- SW3 pad S2: unconnected-(SW3-PadS2) -> GND
- U1 pad 1: unconnected-(U1-PE2-Pad1) -> PE2
- U1 pad 2: unconnected-(U1-PE3-Pad2) -> PE3
- U1 pad 3: unconnected-(U1-PE4-Pad3) -> PE4
- U1 pad 38: unconnected-(U1-PE7-Pad38) -> PE7
- U1 pad 39: unconnected-(U1-PE8-Pad39) -> PE8
- U1 pad 4: unconnected-(U1-PE5-Pad4) -> PE5
- U1 pad 40: unconnected-(U1-PE9-Pad40) -> PE9
- U1 pad 41: unconnected-(U1-PE10-Pad41) -> PE10
- U1 pad 42: unconnected-(U1-PE11-Pad42) -> PE11
- U1 pad 43: unconnected-(U1-PE12-Pad43) -> PE12
- U1 pad 44: unconnected-(U1-PE13-Pad44) -> PE13
- U1 pad 45: unconnected-(U1-PE14-Pad45) -> PE14
- U1 pad 46: unconnected-(U1-PE15-Pad46) -> PE15
- U1 pad 47: unconnected-(U1-PB10-Pad47) -> PB10
- U1 pad 48: unconnected-(U1-PB11-Pad48) -> PB11
- U1 pad 5: unconnected-(U1-PE6-Pad5) -> PE6
- U1 pad 51: unconnected-(U1-PB12-Pad51) -> PB12
- U1 pad 52: unconnected-(U1-PB13-Pad52) -> PB13
- U1 pad 53: unconnected-(U1-PB14-Pad53) -> PB14
- U1 pad 54: unconnected-(U1-PB15-Pad54) -> PB15
- U1 pad 55: unconnected-(U1-PD8-Pad55) -> PD8
- U1 pad 56: unconnected-(U1-PD9-Pad56) -> PD9
- U1 pad 57: unconnected-(U1-PD10-Pad57) -> PD10
- U1 pad 58: unconnected-(U1-PD11-Pad58) -> PD11
- U1 pad 59: unconnected-(U1-PD12-Pad59) -> PD12
- U1 pad 60: unconnected-(U1-PD13-Pad60) -> PD13
- U1 pad 61: unconnected-(U1-PD14-Pad61) -> PD14
- U1 pad 62: unconnected-(U1-PD14-Pad62) -> PD15
- U1 pad 76: DWCLK -> SWCLK
- U1 pad 78: unconnected-(U1-PC10-Pad78) -> PC10
- U1 pad 79: unconnected-(U1-PC11-Pad79) -> PC11
- U1 pad 80: unconnected-(U1-PC12-Pad80) -> PC12
- U1 pad 81: unconnected-(U1-PD0-Pad81) -> PD0
- U1 pad 82: unconnected-(U1-PD1-Pad82) -> PD1
- U1 pad 83: unconnected-(U1-PD2-Pad83) -> PD2
- U1 pad 84: unconnected-(U1-PD3-Pad84) -> PD3
- U1 pad 85: unconnected-(U1-PD4-Pad85) -> PD4
- U1 pad 86: unconnected-(U1-PD5-Pad86) -> PD5
- U1 pad 87: unconnected-(U1-PD6-Pad87) -> PD6
- U1 pad 88: unconnected-(U1-PD7-Pad88) -> PD7
- U1 pad 95: unconnected-(U1-PB8-Pad95) -> PB8
- U1 pad 96: unconnected-(U1-PB9-Pad96) -> PB9
- U1 pad 97: unconnected-(U1-PE0-Pad97) -> PE0
- U1 pad 98: unconnected-(U1-PE1-Pad98) -> PE1
- U2 pad 4: Net-(J3-D+-PadA6) -> Net-(J4-D+-PadA6)
- U2 pad 6: Net-(J3-D--PadA7) -> Net-(J4-D--PadA7)
- U3 pad 4: Net-(J4-D+-PadA6) -> Net-(J5-D+-PadA6)
- U3 pad 6: Net-(J4-D--PadA7) -> Net-(J5-D--PadA7)
- U4 pad 1: Net-(C12-Pad1) -> Net-(C20-Pad1)
- U4 pad 2: Net-(C13-Pad1) -> Net-(C21-Pad1)
- U4 pad 3: Net-(C15-Pad1) -> Net-(C23-Pad1)
- U4 pad 4: Net-(C16-Pad1) -> Net-(C24-Pad1)
Routing:
- net Net-(C24-Pad1): track 0.00 -> 39.9 mm, vias 0 -> 1
- net Net-(C23-Pad1): track 0.00 -> 37.3 mm, vias 0 -> 1
- net Net-(C21-Pad1): track 0.00 -> 34.6 mm, vias 0 -> 1
- net Net-(C20-Pad1): track 0.00 -> 31.4 mm, vias 0 -> 1
- net Earth: track 0.00 -> 26.0 mm
- net StateLED1: track 0.00 -> 16.8 mm
- net StateLED0: track 0.00 -> 16.4 mm
- net P2MDIDN: track 0.00 -> 15.5 mm, vias 0 -> 1
- net P2MDIDP: track 0.00 -> 14.7 mm, vias 0 -> 1
- net P1MDIAP: track 0.00 -> 14.1 mm, vias 0 -> 1
- net P1MDIAN: track 0.00 -> 13.5 mm, vias 0 -> 1
- net P2MDICN: track 0.00 -> 12.8 mm, vias 0 -> 1
- net Eth1_BI_DD+: track 0.00 -> 12.7 mm
- net P2MDIBN: track 0.00 -> 12.6 mm, vias 0 -> 1
- net P1MDIBP: track 0.00 -> 12.5 mm, vias 0 -> 1
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- added copper zone on In2.Cu, net +3.3V
- added copper zone on In1.Cu, net GND
Other:
- outline, holes or cut-outs redrawn
